Commit message: new urdf solid wheels. Trying to debbug wheel and joint problem

File: documents/CAD/Other_Formats/teko_disfunctional/teko.urdf (robot description, URDF)
Before this commit: robot teko, 20 links, 19 joints
Links:
- removed link TEKO_Back_wheel_left
- removed link TEKO_Back_wheel_right
- removed link TEKO_Front_wheel_left
- removed link TEKO_Front_wheel_right
- added link TEKO_WheelBackLeft, mass 0.26591647257735795; collision mesh filename=meshes/TEKO_WheelBackLeft.stl scale=0.001 0.001 0.001; visual mesh filename=meshes/TEKO_WheelBackLeft.stl scale=0.001 0.001 0.001
- added link TEKO_WheelBackRight, mass 0.26593113960593123; collision mesh filename=meshes/TEKO_WheelBackRight.stl scale=0.001 0.001 0.001; visual mesh filename=meshes/TEKO_WheelBackRight.stl scale=0.001 0.001 0.001
- added link TEKO_WheelFrontLeft, mass 0.26591647257735956; collision mesh filename=meshes/TEKO_WheelFrontLeft.stl scale=0.001 0.001 0.001; visual mesh filename=meshes/TEKO_WheelFrontLeft.stl scale=0.001 0.001 0.001
- added link TEKO_WheelFrontRight, mass 0.265931139605929; collision mesh filename=meshes/TEKO_WheelFrontRight.stl scale=0.001 0.001 0.001; visual mesh filename=meshes/TEKO_WheelFrontRight.stl scale=0.001 0.001 0.001
Joints:
- removed joint TEKO_Chassi_Back_wheel_left
- removed joint TEKO_Chassi_Back_wheel_right
- removed joint TEKO_Chassi_Front_wheel_left
- removed joint TEKO_Chassi_Front_wheel_right
- added joint TEKO_Chassi_JointWheelBackLeft: type continuous, parent TEKO_Chassi, child TEKO_WheelBackLeft, origin xyz=-0.12605402 0.015 -0.09565 rpy=-1.5707963267948966 -0.0 0.0, axis 0.0 0.0 1.0
- added joint TEKO_Chassi_JointWheelBackRight: type continuous, parent TEKO_Chassi, child TEKO_WheelBackRight, origin xyz=-0.12605402 -0.149 -0.09565 rpy=1.5707963267948966 -0.0 0.0, axis 0.0 0.0 -1.0
- added joint TEKO_Chassi_JointWheelFrontLeft: type continuous, parent TEKO_Chassi, child TEKO_WheelFrontLeft, origin xyz=0.04784598000000001 0.015 -0.09565 rpy=-1.5707963267948966 -0.0 0.0, axis 0.0 0.0 1.0
- added joint TEKO_Chassi_JointWheelFrontRight: type continuous, parent TEKO_Chassi, child TEKO_WheelFrontRight, origin xyz=0.04784598000000001 -0.149 -0.09565 rpy=1.5707963267948966 -0.0 0.0, axis 0.0 0.0 -1.0
- joint TEKO_LidarBase_JointLidar: axis (none) -> 0.0 -0.0 1.0; type fixed -> continuous
