Commit message: v1.6_finally_new_going_forward

File: documents/CAD/Other_Formats/teko/teko.urdf (robot description, URDF)
Before this commit: robot teko_urdf, 19 links, 18 joints
Links:
- removed link TEKO_BoardSupport-1
- removed link TEKO_ChassiUpper
- removed link TEKO_ConnectorFront
- added link TEKO_ArucoSuppor, mass 2.3849467441322254; collision mesh filename=meshes/TEKO_ArucoSuppor.stl scale=0.001 0.001 0.001; visual mesh filename=meshes/TEKO_ArucoSuppor.stl scale=0.001 0.001 0.001
- added link TEKO_Chassi, mass 0.8515121958050561; collision mesh filename=meshes/TEKO_Chassi.stl scale=0.001 0.001 0.001; visual mesh filename=meshes/TEKO_Chassi.stl scale=0.001 0.001 0.001
- added link TEKO_ConnectorMale, mass 0.5231990984505147; collision mesh filename=meshes/TEKO_ConnectorMale.stl scale=0.001 0.001 0.001; visual mesh filename=meshes/TEKO_ConnectorMale.stl scale=0.001 0.001 0.001
- added link TEKO_ConnectorPin, mass 0.06016190580093297; collision mesh filename=meshes/TEKO_ConnectorPin.stl scale=0.001 0.001 0.001; visual mesh filename=meshes/TEKO_ConnectorPin.stl scale=0.001 0.001 0.001
- link TEKO_Body: mass 0.8515121958050561 -> 2.95242908958936
Joints:
- removed joint TEKO_BoardSupport-1_JointArucoGlass
- removed joint TEKO_Body_BackLeft
- removed joint TEKO_Body_BackRight
- removed joint TEKO_Body_FrontLeft
- removed joint TEKO_Body_FrontRight
- removed joint TEKO_Body_JointMotorLeft
- removed joint TEKO_Body_JointMotorRight
- removed joint TEKO_ChassiUpper_JointArucoSupport
- removed joint TEKO_ChassiUpper_JointBackWall
- removed joint TEKO_ChassiUpper_JointBoards
- removed joint TEKO_ChassiUpper_JointBothChassis
- removed joint TEKO_ChassiUpper_JointConnectorFront
- removed joint TEKO_ChassiUpper_JointConnectorRear
- removed joint TEKO_ChassiUpper_JointGlassUnder
- removed joint TEKO_ChassiUpper_JointLidarSupport
- removed joint TEKO_ChassiUpper_JointRoof
- removed joint TEKO_WallBack_JointCamera
- added joint TEKO_ArucoSuppor_ArucoGlass: type fixed, parent TEKO_ArucoSuppor, child TEKO_GlassAruco, origin xyz=-0.021999999999999992 -0.019000000000000003 0.00699999 rpy=0.0 -0.0 0.0
- added joint TEKO_Body_ArucoSupport: type fixed, parent TEKO_Body, child TEKO_ArucoSuppor, origin xyz=0.17250000000000001 0.067 -0.0575 rpy=0.0 -0.0 0.0
- added joint TEKO_Body_BackWall: type fixed, parent TEKO_Body, child TEKO_WallBack, origin xyz=-0.168625 0.0 -0.0575 rpy=0.0 -0.0 0.0
- added joint TEKO_Body_BoardSupport: type fixed, parent TEKO_Body, child TEKO_BoardSupport, origin xyz=0.0327 0.0668 -0.0575 rpy=-1.5707963267948966 -1.3559975873284387e-14 1.570796326794902
- added joint TEKO_Body_ConnectorFront: type fixed, parent TEKO_Body, child TEKO_ConnectorMale, origin xyz=0.17250000000000001 0.0 -0.057999999999999996 rpy=-1.5707963267948966 -9.310046328093557e-17 -1.5707963267948966
- added joint TEKO_Body_ConnectorRear: type fixed, parent TEKO_Body, child TEKO_ConnectorRear, origin xyz=-0.17250000000000001 0.0 -0.057999999999999996 rpy=1.5707963267948966 9.310046328093557e-17 -1.5707963267948977
- added joint TEKO_Body_FullBody: type fixed, parent TEKO_Body, child TEKO_Chassi, origin xyz=0.0327 0.0668 -0.0575 rpy=0.0 -0.0 0.0
- added joint TEKO_Body_GlassUnder: type fixed, parent TEKO_Body, child TEKO_GlassBase, origin xyz=-0.17250000000000001 0.067 -0.07730000000000001 rpy=3.141592653589793 -0.0 1.5707963267948966
- added joint TEKO_Body_LidarSupport: type fixed, parent TEKO_Body, child TEKO_LidarBase, origin xyz=0.17250000000000001 -0.0477 0.057999999999999996 rpy=-1.5707963267948966 -1.5707963267948966 0
- added joint TEKO_Body_Roof: type fixed, parent TEKO_Body, child TEKO_Roof, origin xyz=0.17250000000000001 -0.067 0.07730000000000001 rpy=0.0 -0.0 -1.5707963267948966
- added joint TEKO_Chassi_JointWheelBackLeft: type continuous, parent TEKO_Chassi, child TEKO_WheelBackLeft, origin xyz=-0.12605402 0.015 -0.09565 rpy=-1.5707963267948966 -0.0 0.0, axis 0.0 0.0 1.0
- added joint TEKO_Chassi_JointWheelBackRight: type continuous, parent TEKO_Chassi, child TEKO_WheelBackRight, origin xyz=-0.12605402 -0.149 -0.09565 rpy=1.5707963267948966 -0.0 0.0, axis 0.0 0.0 1.0
- added joint TEKO_Chassi_JointWheelFrontLeft: type continuous, parent TEKO_Chassi, child TEKO_WheelFrontLeft, origin xyz=0.04784598000000001 0.015 -0.09565 rpy=-1.5707963267948966 -0.0 0.0, axis 0.0 0.0 1.0
- added joint TEKO_Chassi_JointWheelFrontRight: type continuous, parent TEKO_Chassi, child TEKO_WheelFrontRight, origin xyz=0.04784598000000001 -0.149 -0.09565 rpy=1.5707963267948966 -0.0 0.0, axis 0.0 0.0 1.0
- added joint TEKO_Chassi_MotorLeft: type fixed, parent TEKO_Chassi, child TEKO_MotorRight-1, origin xyz=-0.12605402 0.005 -0.09565 rpy=1.5707963267948963 -0.0 0.0
- added joint TEKO_Chassi_MotorRight: type fixed, parent TEKO_Chassi, child TEKO_MotorRight, origin xyz=-0.12605402 -0.13899999999999998 -0.09565 rpy=-1.5707963267948963 -0.0 0.0
- added joint TEKO_ConnectorMale_JointPin: type fixed, parent TEKO_ConnectorMale, child TEKO_ConnectorPin, origin xyz=-8.617000000000059e-05 0.006360130000000002 0.05649999999999999 rpy=3.141592653589793 -0.0 -1.5707963267948966
- added joint TEKO_WallBack_Camera: type fixed, parent TEKO_WallBack, child TEKO_Camera, origin xyz=-0.0030999999999999873 0.0 0.11499528 rpy=1.5707963267948966 -0.0 -1.570796326794897

Commit message: Add Optuna training, fix wheel axis in URDF, update rewards and curriculum

File: documents/CAD/Other_Formats/teko/teko.urdf (robot description, URDF)
Before this commit: robot teko_urdf, 20 links, 19 joints
Joints:
- joint TEKO_Chassi_JointWheelBackRight: axis 0.0 0.0 1.0 -> 0.0 0.0 -1.0
- joint TEKO_Chassi_JointWheelFrontRight: axis 0.0 0.0 1.0 -> 0.0 0.0 -1.0

Commit message: URDF changes

File: documents/CAD/Other_Formats/teko/teko.urdf (robot description, URDF)
Before this commit: robot teko, 20 links, 19 joints
Joints:
- joint TEKO_Chassi_Back_wheel_left: axis 0.0 0.0 -1.0 -> 0.0 0.0 1.0
- joint TEKO_Chassi_Back_wheel_right: axis 0.0 0.0 1.0 -> 0.0 0.0 -1.0
- joint TEKO_Chassi_Front_wheel_left: axis 0.0 0.0 -1.0 -> 0.0 0.0 1.0
- joint TEKO_Chassi_Front_wheel_right: axis 0.0 0.0 1.0 -> 0.0 0.0 -1.0

Commit message: rotation vai -90

File: documents/CAD/Other_Formats/teko/teko.urdf (robot description, URDF)
Before this commit: robot teko, 20 links, 19 joints
Links:
- removed link TEKO_Back_wheel_left
- removed link TEKO_Back_wheel_right
- removed link TEKO_Front_wheel_left
- removed link TEKO_Front_wheel_right
- added link TEKO_WheelBackLeft, mass 0.26591647257735795; collision mesh filename=meshes/TEKO_WheelBackLeft.stl scale=0.001 0.001 0.001; visual mesh filename=meshes/TEKO_WheelBackLeft.stl scale=0.001 0.001 0.001
- added link TEKO_WheelBackRight, mass 0.26593113960593123; collision mesh filename=meshes/TEKO_WheelBackRight.stl scale=0.001 0.001 0.001; visual mesh filename=meshes/TEKO_WheelBackRight.stl scale=0.001 0.001 0.001
- added link TEKO_WheelFrontLeft, mass 0.26591647257735956; collision mesh filename=meshes/TEKO_WheelFrontLeft.stl scale=0.001 0.001 0.001; visual mesh filename=meshes/TEKO_WheelFrontLeft.stl scale=0.001 0.001 0.001
- added link TEKO_WheelFrontRight, mass 0.265931139605929; collision mesh filename=meshes/TEKO_WheelFrontRight.stl scale=0.001 0.001 0.001; visual mesh filename=meshes/TEKO_WheelFrontRight.stl scale=0.001 0.001 0.001
Joints:
- removed joint TEKO_Chassi_Back_wheel_left
- removed joint TEKO_Chassi_Back_wheel_right
- removed joint TEKO_Chassi_Front_wheel_left
- removed joint TEKO_Chassi_Front_wheel_right
- added joint TEKO_Chassi_JointWheelBackLeft: type continuous, parent TEKO_Chassi, child TEKO_WheelBackLeft, origin xyz=-0.12605402 0.015 -0.09565 rpy=-1.5707963267948966 -0.0 0.0, axis 0.0 0.0 1.0
- added joint TEKO_Chassi_JointWheelBackRight: type continuous, parent TEKO_Chassi, child TEKO_WheelBackRight, origin xyz=-0.12605402 -0.149 -0.09565 rpy=1.5707963267948966 -0.0 0.0, axis 0.0 0.0 1.0
- added joint TEKO_Chassi_JointWheelFrontLeft: type continuous, parent TEKO_Chassi, child TEKO_WheelFrontLeft, origin xyz=0.04784598000000001 0.015 -0.09565 rpy=-1.5707963267948966 -0.0 0.0, axis 0.0 0.0 1.0
- added joint TEKO_Chassi_JointWheelFrontRight: type continuous, parent TEKO_Chassi, child TEKO_WheelFrontRight, origin xyz=0.04784598000000001 -0.149 -0.09565 rpy=1.5707963267948966 -0.0 0.0, axis 0.0 0.0 1.0
- joint TEKO_LidarBase_JointLidar: axis (none) -> 0.0 -0.0 1.0; type fixed -> continuous
